Commit message: added "world_link" for fixing the robot

File: arm_description/urdf/arm.urdf.xacro (robot description, xacro)
@@ -4,4 +4,11 @@
     <color rgba="1 0 0 1"/>
   </material>
+<!-- Used for fixing robot-->
+  <link name="world"/>
+  <joint name="base_link_joint" type="fixed">
+      <origin rpy="0.0 0 0" xyz="0 0 0"/>
+      <parent link="world"/>
+      <child link="base_link"/>
+  </joint>
   <link name="base_link">
     <visual>
